Commit message: Update the DR-SPAAM to use KD-Tree Masking for map nased LiDAR masking. And update the LiDAR sensor to match S2L.

File: src/smrr_description/urdf/lidar.urdf.xacro (robot description, xacro)
@@ -3,7 +3,7 @@
 	<link name="rplidar_link">
         <inertial>
-			<mass value="1e-5"/>
+			<mass value="0.1"/>
 			<origin xyz="0 0 0" rpy="0 0 0"/>
-			<inertia ixx="1e-6" ixy="0" ixz="0" iyy="1e-6" iyz="0" izz="1e-6"/>
+			<inertia ixx="0.001" ixy="0" ixz="0" iyy="0.001" iyz="0" izz="0.001"/>
 		</inertial>
 		<visual>
@@ -35,5 +35,5 @@
                 <scan>
                     <horizontal>
-                        <samples>400</samples>
+                        <samples>2133</samples>
                         <resolution>1</resolution>
                         <min_angle>-2.0943</min_angle>
@@ -42,6 +42,6 @@
                 </scan>
                 <range>
-                    <min>0.15</min>
-                    <max>12.0</max> <!--6.0 -->
+                    <min>0.05</min>
+                    <max>18.0</max> <!--6.0 -->
                     <resolution>0.01</resolution>
                 </range>
@@ -49,5 +49,5 @@
                     <type>gaussian</type>
                     <mean>0.0</mean>
-                    <stddev>0.01</stddev>
+                    <stddev>0.015</stddev>
                 </noise>
             </ray>

Commit message: Added elevator moving direction detection before boarding the elevator.

File: src/smrr_description/urdf/lidar.urdf.xacro (robot description, xacro)
@@ -23,5 +23,5 @@
     </link>
 	<joint name="rplidar_joint" type="fixed">
-		<origin xyz="0.23 0 0.1874" rpy="0 0 0 "/>
+		<origin xyz="0.24 0 0.1874" rpy="0 0 0 "/>
 		<parent link="base_link"/>
 		<child link="rplidar_link"/>

Commit message: Robot branch updates for bringup, controller, localization, and navigation

File: src/smrr_description/urdf/lidar.urdf.xacro (robot description, xacro)
@@ -23,5 +23,5 @@
     </link>
 	<joint name="rplidar_joint" type="fixed">
-		<origin xyz="0.23 0 0.001" rpy="0 0 0 "/>
+		<origin xyz="0.24 0  0.1874" rpy="0 0 0 "/>
 		<parent link="base_link"/>
 		<child link="rplidar_link"/>

Commit message: Selective merge from robot-branch (exclude zed/sllidar packages)

File: src/smrr_description/urdf/lidar.urdf.xacro (robot description, xacro)
@@ -3,7 +3,7 @@
 	<link name="rplidar_link">
         <inertial>
-			<mass value="0.1"/>
+			<mass value="1e-5"/>
 			<origin xyz="0 0 0" rpy="0 0 0"/>
-			<inertia ixx="0.001" ixy="0" ixz="0" iyy="0.001" iyz="0" izz="0.001"/>
+			<inertia ixx="1e-6" ixy="0" ixz="0" iyy="1e-6" iyz="0" izz="1e-6"/>
 		</inertial>
 		<visual>
@@ -23,5 +23,5 @@
     </link>
 	<joint name="rplidar_joint" type="fixed">
-		<origin xyz="0.24 0 0.1874" rpy="0 0 0 "/>
+		<origin xyz="0.24 0  0.1874" rpy="0 0 0 "/>
 		<parent link="base_link"/>
 		<child link="rplidar_link"/>
@@ -31,9 +31,9 @@
             <pose>0 0 0 0 0 0</pose>
             <visualize>true</visualize>
-            <update_rate>10</update_rate>
+            <update_rate>30</update_rate>
             <ray>
                 <scan>
                     <horizontal>
-                        <samples>2133</samples>
+                        <samples>400</samples>
                         <resolution>1</resolution>
                         <min_angle>-2.0943</min_angle>
@@ -42,6 +42,6 @@
                 </scan>
                 <range>
-                    <min>0.05</min>
-                    <max>18.0</max> <!--6.0 -->
+                    <min>0.15</min>
+                    <max>12.0</max> <!--6.0 -->
                     <resolution>0.01</resolution>
                 </range>
@@ -49,5 +49,5 @@
                     <type>gaussian</type>
                     <mean>0.0</mean>
-                    <stddev>0.015</stddev>
+                    <stddev>0.01</stddev>
                 </noise>
             </ray>
