Commit message: Updated the lidar range to 240 dgrees, dynamic costmap inflation

File: src/smrr_description/urdf/right_hand.urdf.xacro (robot description, xacro)
@@ -47,5 +47,4 @@
     name="shoulder_r_joint"
     type="fixed">
-    <!-- type="revolute" -->
     <origin
       xyz="0.0025 -0.17549 1.13"
@@ -55,11 +54,4 @@
     <child
       link="shoulder_r_link" />
-    <axis
-      xyz="0 0 1" />
-    <limit
-      lower="0"
-      upper="${0.5*PI}"
-      effort="0"
-      velocity="0" />
   </joint>
   <link
@@ -108,5 +100,4 @@
     name="bicep_r_joint"
     type="fixed">
-    <!-- type="revolute" -->
     <origin
       xyz="-0.00044422 -0.12491 -0.0013064"
@@ -116,11 +107,4 @@
     <child
       link="bicep_r_link" />
-    <axis
-      xyz="0 0 1" />
-    <limit
-      lower="${-0.25*PI}"
-      upper="${0.25*PI}"
-      effort="0"
-      velocity="0" />
   </joint>
   <link
@@ -169,5 +153,4 @@
     name="elbow_r_joint"
     type="fixed">
-    <!-- type="revolute" -->
     <origin
       xyz="0.010186 -0.0047446 0.14136"
@@ -177,11 +160,4 @@
     <child
       link="elbow_r_link" />
-    <axis
-      xyz="-0.06561 0.035186 0.99722" />
-    <limit
-      lower="0"
-      upper="${0.5*PI}"
-      effort="0"
-      velocity="0" />
   </joint>
   <link
@@ -230,5 +206,4 @@
     name="wrist_r_joint"
     type="fixed">
-    <!-- type="revolute" -->
     <origin
       xyz="0.057171 -0.23705 0.0080661"
@@ -238,11 +213,4 @@
     <child
       link="wrist_r_link" />
-    <axis
-      xyz="0 0 1" />
-    <limit
-      lower="${-0.25*PI}"
-      upper="${0.25*PI}"
-      effort="0"
-      velocity="0" />
   </joint>
   <link name="eef_r_link" />
