Commit message: Add docking functionality with configuration and launch files
- Updated model paths in sim_world.world for docking station and Apriltag.
- Changed world file reference in gazebo_classic_controllers.launch.py.
- Added rear camera configuration in camera.urdf.xacro for docking.
- Updated map server parameters in smrr_nav_params.yaml.
- Created docking.yaml with parameters for docking server.
- Implemented docking_bringup.launch.py to launch docking server and related nodes.
- Added package.xml and setup files for smrr_docking package.
- Developed publish_state_dock_pose.py to publish static dock pose.
- Added copyright and flake8 tests.

File: src/smrr_description/urdf/camera.urdf.xacro (robot description, xacro)
@@ -136,3 +136,140 @@
         </sensor>
     </gazebo>
+    <!-- ============================================ -->
+    <!-- REAR CAMERA FOR DOCKING                     -->
+    <!-- ============================================ -->
+    <!-- Rear Camera Mount (facing backward for docking) -->
+    <joint name="rear_camera_joint" type="fixed">
+        <origin xyz="-0.08 0 0.15" rpy="0 0 ${pi}"/>  <!-- Mounted at back, rotated 180° -->
+        <parent link="base_link"/>
+        <child link="rear_camera_link"/>
+    </joint>
+    <link name="rear_camera_link">
+        <inertial>
+            <mass value="0.16140"/>
+            <origin xyz="0 0 0"/>
+            <inertia
+                ixx="0.0003947" ixy="0.0" ixz="3.3365e-8"
+                iyy="2.417e-5" iyz="0.0"
+                izz="0.0003973"/>
+        </inertial>
+        <visual>
+            <origin xyz="0 0 0" rpy="0 0 1.57"/>
+            <geometry>
+                <mesh filename="package://smrr_description/meshes/ZED2i.stl" scale="0.001 0.001 0.001"/>
+            </geometry>
+        </visual>
+        <collision>
+            <origin xyz="0 0 0" rpy="0 0 1.57"/>
+            <geometry>
+                <mesh filename="package://smrr_description/meshes/ZED2i.stl" scale="0.001 0.001 0.001"/>
+            </geometry>
+        </collision>
+    </link>
+    <!-- Rear Left Camera -->
+    <joint name="rear_left_camera_joint" type="fixed">
+        <parent link="rear_camera_link"/>
+        <child link="rear_left_camera_link"/>
+        <origin xyz="0 0.06 0" rpy="0 0 0"/>
+    </joint>
+    <link name="rear_left_camera_link"></link>
+    <joint name="rear_left_camera_optical_joint" type="fixed">
+        <parent link="rear_left_camera_link"/>
+        <child link="rear_left_camera_link_optical"/>
+        <origin xyz="0 0 0" rpy="${-pi/2} 0 ${-pi/2}"/>
+    </joint>
+    <link name="rear_left_camera_link_optical"></link>
+    <!-- Rear Right Camera -->
+    <joint name="rear_right_camera_joint" type="fixed">
+        <parent link="rear_camera_link"/>
+        <child link="rear_right_camera_link"/>
+        <origin xyz="0 -0.06 0" rpy="0 0 0"/>
+    </joint>
+    <link name="rear_right_camera_link"></link>
+    <joint name="rear_right_camera_optical_joint" type="fixed">
+        <parent link="rear_right_camera_link"/>
+        <child link="rear_right_camera_link_optical"/>
+        <origin xyz="0 0 0" rpy="${-pi/2} 0 ${-pi/2}"/>
+    </joint>
+    <link name="rear_right_camera_link_optical"></link>
+    <!-- Rear Camera Gazebo Sensors -->
+    <gazebo reference="rear_left_camera_link">
+        <material>Gazebo/Blue</material>  <!-- Different color to distinguish from front camera -->
+        <!-- Rear Camera Raw Images -->
+        <sensor name="zed2_rear_left_raw_camera" type="camera">
+            <pose> 0 0 0 0 0 0 </pose>
+            <visualize>true</visualize>
+            <always_on>true</always_on>
+            <update_rate>15</update_rate>
+            <camera>
+                <horizontal_fov>1.7633</horizontal_fov>
+                <image>
+                    <format>R8G8B8</format>
+                    <width>1280</width>
+                    <height>720</height>
+                </image>
+                <clip>
+                    <near>0.1</near>
+                    <far>300</far>
+                </clip>
+                <noise>
+                    <type>gaussian</type>
+                    <mean>0.0</mean>
+                    <stddev>0.007</stddev>
+                </noise>
+                <distortion>
+                    <!-- Same ZED2 distortion parameters -->
+                    <k1>-0.043693598</k1>
+                    <k2>0.0146164996</k2>
+                    <p1>-0.006573319</p1>
+                    <p2>-0.000216900</p2>
+                    <k3>0.000084328</k3>
+                    <center>0.5 0.5</center>
+                </distortion>
+            </camera>
+            <plugin name="rear_camera_controller" filename="libgazebo_ros_camera.so">
+                <cameraName>zed2_rear/zed_node/left_raw</cameraName>
+                <imageTopicName>image_raw_color</imageTopicName>
+                <cameraInfoTopicName>camera_info</cameraInfoTopicName>
+                <frameName>rear_left_camera_link_optical</frameName>
+                <distortionK1>-0.043693598</distortionK1>
+                <distortionK2>0.0146164996</distortionK2>
+                <distortionT1>-0.006573319</distortionT1>
+                <distortionT2>-0.000216900</distortionT2>
+                <distortionK3>0.000084328</distortionK3>
+                <CxPrime>648.5</CxPrime>
+                <Cx>648.5</Cx>
+                <Cy>366.8340148925781</Cy>
+                <hackBaseline>0.0</hackBaseline>
+            </plugin>
+        </sensor>
+        <!-- Rear Camera Depth Sensor -->
+        <sensor name="zed2_rear_left_camera" type="depth">
+            <visualize>true</visualize>
+            <always_on>true</always_on>
+            <update_rate>15</update_rate>
+            <camera name="zed2_rear_left">
+                <horizontal_fov>1.7633</horizontal_fov>
+                <image>
+                    <format>R8G8B8</format>
+                    <width>1280</width>
+                    <height>720</height>
+                </image>
+                <clip>
+                    <near>0.1</near>
+                    <far>300</far>
+                </clip>
+                <noise>
+                    <type>gaussian</type>
+                    <mean>0.0</mean>
+                    <stddev>0.007</stddev>
+                </noise>
+            </camera>
+            <plugin name="rear_depth_camera_controller" filename="libgazebo_ros_camera.so">
+                <frame_name>rear_left_camera_link_optical</frame_name>
+                <min_depth>0.1</min_depth>
+                <max_depth>100.0</max_depth>
+            </plugin>
+        </sensor>
+    </gazebo>
 </robot>

Commit message: Successfully docked with the physical robot. Need to adjust the final docking parameters.

File: src/smrr_description/urdf/camera.urdf.xacro (robot description, xacro)
@@ -136,3 +136,140 @@
         </sensor>
     </gazebo>
+    <!-- ============================================ -->
+    <!-- REAR CAMERA FOR DOCKING                     -->
+    <!-- ============================================ -->
+    <!-- Rear Camera Mount (facing backward for docking) -->
+    <joint name="rear_camera_joint" type="fixed">
+        <origin xyz="-0.12 0 0.43" rpy="0 0 ${pi}"/>  <!-- Mounted at back, rotated 180° -->
+        <parent link="base_link"/>
+        <child link="rear_camera_link"/>
+    </joint>
+    <link name="rear_camera_link">
+        <inertial>
+            <mass value="0.16140"/>
+            <origin xyz="0 0 0"/>
+            <inertia
+                ixx="0.0003947" ixy="0.0" ixz="3.3365e-8"
+                iyy="2.417e-5" iyz="0.0"
+                izz="0.0003973"/>
+        </inertial>
+        <visual>
+            <origin xyz="0 0 0" rpy="0 0 1.57"/>
+            <geometry>
+                <mesh filename="package://smrr_description/meshes/ZED2i.stl" scale="0.001 0.001 0.001"/>
+            </geometry>
+        </visual>
+        <collision>
+            <origin xyz="0 0 0" rpy="0 0 1.57"/>
+            <geometry>
+                <mesh filename="package://smrr_description/meshes/ZED2i.stl" scale="0.001 0.001 0.001"/>
+            </geometry>
+        </collision>
+    </link>
+    <!-- Rear Left Camera -->
+    <joint name="rear_left_camera_joint" type="fixed">
+        <parent link="rear_camera_link"/>
+        <child link="rear_left_camera_link"/>
+        <origin xyz="0 0.06 0" rpy="0 0 0"/>
+    </joint>
+    <link name="rear_left_camera_link"></link>
+    <joint name="rear_left_camera_optical_joint" type="fixed">
+        <parent link="rear_left_camera_link"/>
+        <child link="rear_left_camera_link_optical"/>
+        <origin xyz="0 0 0" rpy="${-pi/2} 0 ${-pi/2}"/>
+    </joint>
+    <link name="rear_left_camera_link_optical"></link>
+    <!-- Rear Right Camera -->
+    <joint name="rear_right_camera_joint" type="fixed">
+        <parent link="rear_camera_link"/>
+        <child link="rear_right_camera_link"/>
+        <origin xyz="0 -0.06 0" rpy="0 0 0"/>
+    </joint>
+    <link name="rear_right_camera_link"></link>
+    <joint name="rear_right_camera_optical_joint" type="fixed">
+        <parent link="rear_right_camera_link"/>
+        <child link="rear_right_camera_link_optical"/>
+        <origin xyz="0 0 0" rpy="${-pi/2} 0 ${-pi/2}"/>
+    </joint>
+    <link name="rear_right_camera_link_optical"></link>
+    <!-- Rear Camera Gazebo Sensors -->
+    <gazebo reference="rear_left_camera_link">
+        <material>Gazebo/Blue</material>  <!-- Different color to distinguish from front camera -->
+        <!-- Rear Camera Raw Images -->
+        <sensor name="zed2_rear_left_raw_camera" type="camera">
+            <pose> 0 0 0 0 0 0 </pose>
+            <visualize>false</visualize>
+            <always_on>true</always_on>
+            <update_rate>15</update_rate>
+            <camera>
+                <horizontal_fov>1.7633</horizontal_fov>
+                <image>
+                    <format>R8G8B8</format>
+                    <width>1280</width>
+                    <height>720</height>
+                </image>
+                <clip>
+                    <near>0.1</near>
+                    <far>300</far>
+                </clip>
+                <noise>
+                    <type>gaussian</type>
+                    <mean>0.0</mean>
+                    <stddev>0.007</stddev>
+                </noise>
+                <distortion>
+                    <!-- Same ZED2 distortion parameters -->
+                    <k1>-0.043693598</k1>
+                    <k2>0.0146164996</k2>
+                    <p1>-0.006573319</p1>
+                    <p2>-0.000216900</p2>
+                    <k3>0.000084328</k3>
+                    <center>0.5 0.5</center>
+                </distortion>
+            </camera>
+            <plugin name="rear_camera_controller" filename="libgazebo_ros_camera.so">
+                <cameraName>zed2_rear/zed_node/left_raw</cameraName>
+                <imageTopicName>image_raw_color</imageTopicName>
+                <cameraInfoTopicName>camera_info</cameraInfoTopicName>
+                <frameName>rear_left_camera_link_optical</frameName>
+                <distortionK1>-0.043693598</distortionK1>
+                <distortionK2>0.0146164996</distortionK2>
+                <distortionT1>-0.006573319</distortionT1>
+                <distortionT2>-0.000216900</distortionT2>
+                <distortionK3>0.000084328</distortionK3>
+                <CxPrime>648.5</CxPrime>
+                <Cx>648.5</Cx>
+                <Cy>366.8340148925781</Cy>
+                <hackBaseline>0.0</hackBaseline>
+            </plugin>
+        </sensor>
+        <!-- Rear Camera Depth Sensor -->
+        <sensor name="zed2_rear_left_camera" type="depth">
+            <visualize>false</visualize>
+            <always_on>true</always_on>
+            <update_rate>15</update_rate>
+            <camera name="zed2_rear_left">
+                <horizontal_fov>1.7633</horizontal_fov>
+                <image>
+                    <format>R8G8B8</format>
+                    <width>1280</width>
+                    <height>720</height>
+                </image>
+                <clip>
+                    <near>0.1</near>
+                    <far>300</far>
+                </clip>
+                <noise>
+                    <type>gaussian</type>
+                    <mean>0.0</mean>
+                    <stddev>0.007</stddev>
+                </noise>
+            </camera>
+            <plugin name="rear_depth_camera_controller" filename="libgazebo_ros_camera.so">
+                <frame_name>rear_left_camera_link_optical</frame_name>
+                <min_depth>0.1</min_depth>
+                <max_depth>100.0</max_depth>
+            </plugin>
+        </sensor>
+    </gazebo>
 </robot>

Commit message: Implemeneted the smrr_crowdnav package for human tracking using YOLO based and lidar based approach. The name of the package needed to be changed.

File: src/smrr_description/urdf/camera.urdf.xacro (robot description, xacro)
@@ -66,5 +66,5 @@
             <update_rate>15</update_rate>
             <camera>
-                <horizontal_fov>1.7633</horizontal_fov>
+                <horizontal_fov>1.9199</horizontal_fov>
                 <image>
                     <format>R8G8B8</format>
@@ -113,5 +113,5 @@
             <update_rate>15</update_rate>
             <camera name="zed2_left">
-                <horizontal_fov>1.7633</horizontal_fov>
+                <horizontal_fov>1.9199</horizontal_fov>
                 <image>
                     <format>R8G8B8</format>
@@ -203,5 +203,5 @@
             <update_rate>15</update_rate>
             <camera>
-                <horizontal_fov>1.7633</horizontal_fov>
+                <horizontal_fov>1.9199</horizontal_fov>
                 <image>
                     <format>R8G8B8</format>
@@ -236,5 +236,5 @@
             <update_rate>15</update_rate>
             <camera name="zed2_rear_left">
-                <horizontal_fov>1.7633</horizontal_fov>
+                <horizontal_fov>1.9199</horizontal_fov>
                 <image>
                     <format>R8G8B8</format>

File: src/smrr_description/urdf/lidar.urdf.xacro (robot description, xacro)
@@ -23,5 +23,5 @@
     </link>
 	<joint name="rplidar_joint" type="fixed">
-		<origin xyz="0.23 0 0.001" rpy="0 0 0 "/>
+		<origin xyz="0.23 0 0.1874" rpy="0 0 0 "/>
 		<parent link="base_link"/>
 		<child link="rplidar_link"/>

File: src/smrr_description/urdf/mobile_base.urdf.xacro (robot description, xacro)
@@ -20,12 +20,12 @@
         rpy="0 0 0" />
       <mass
-        value="17.0" />
-      <inertia
-        ixx="1.5"
+        value="10.0" />
+      <inertia
+        ixx="1.0"
         ixy="0.0"
         ixz="0.0"
-        iyy="1.5"
+        iyy="1.0"
         iyz="0.0"
-        izz="1.0" />
+        izz="0.8" />
     </inertial>
     <visual>
@@ -57,15 +57,15 @@
     <inertial>
       <origin
-        xyz="3.04623488683875E-06 6.72391256367755E-06 -0.0311105168378413"
-        rpy="0 0 0" />
-      <mass
-        value="0.989823090734283" />
-      <inertia
-        ixx="0.00167921032012111"
-        ixy="6.53172867821882E-09"
-        ixz="-1.64665780609969E-07"
-        iyy="0.0016792904624912"
-        iyz="-3.63464523309006E-07"
-        izz="0.00288690083815089" />
+        xyz="0 0 0"
+        rpy="0 0 0" />
+      <mass
+        value="1.5" />
+      <inertia
+        ixx="0.0025"
+        ixy="0.0"
+        ixz="0.0"
+        iyy="0.0025"
+        iyz="0.0"
+        izz="0.0044" />
     </inertial>
     <visual>
@@ -124,5 +124,5 @@
     <axis
       xyz="0 0 1" />
-    <dynamics damping="0.1" friction="0.01"/>
+    <dynamics damping="0.0" friction="0.0"/>
   </joint>
   <link
@@ -130,15 +130,15 @@
     <inertial>
       <origin
-        xyz="-8.38679888204297E-07 7.3339732202804E-06 0.0311105168378413"
-        rpy="0 0 0" />
-      <mass
-        value="0.989823090734282" />
-      <inertia
-        ixx="0.00167926061595776"
-        ixy="-1.12032618333546E-08"
-        ixz="-4.53352691396202E-08"
-        iyy="0.00167924016665455"
-        iyz="3.96441663275016E-07"
-        izz="0.0028869008381509" />
+        xyz="0 0 0"
+        rpy="0 0 0" />
+      <mass
+        value="1.5" />
+      <inertia
+        ixx="0.0025"
+        ixy="0.0"
+        ixz="0.0"
+        iyy="0.0025"
+        iyz="0.0"
+        izz="0.0044" />
     </inertial>
     <visual>
@@ -199,5 +199,5 @@
       <axis
         xyz="0 0 1" />
-      <dynamics damping="0.1" friction="0.01"/>
+      <dynamics damping="0.0" friction="0.0"/>
   </joint>
   <!-- <link
@@ -291,15 +291,15 @@
     <inertial>
       <origin
-        xyz="0 0 -0.0025"
-        rpy="0 0 0" />
-      <mass
-        value="0.0335103216382911" />
-      <inertia
-        ixx="5.36165146212658E-06"
-        ixy="0"
-        ixz="-9.4039548065783E-38"
-        iyy="5.36165146212658E-06"
-        iyz="0"
-        izz="5.36165146212658E-06" />
+        xyz="0 0 0"
+        rpy="0 0 0" />
+      <mass
+        value="0.5" />
+      <inertia
+        ixx="0.0001"
+        ixy="0.0"
+        ixz="0.0"
+        iyy="0.0001"
+        iyz="0.0"
+        izz="0.0001" />
     </inertial>
     <visual>
@@ -350,5 +350,5 @@
     type="fixed">
     <origin
-      xyz="0.245 0 -0.04"
+      xyz="0.245 0 -0.0414"
       rpy="0 0 0" />
     <parent
@@ -364,15 +364,15 @@
     <inertial>
       <origin
-        xyz="0 0 -0.0025"
-        rpy="0 0 0" />
-      <mass
-        value="0.0335103216382911" />
-      <inertia
-        ixx="5.36165146212658E-06"
-        ixy="0"
-        ixz="-9.4039548065783E-38"
-        iyy="5.36165146212658E-06"
-        iyz="0"
-        izz="5.36165146212658E-06" />
+        xyz="0 0 0"
+        rpy="0 0 0" />
+      <mass
+        value="0.5" />
+      <inertia
+        ixx="0.0001"
+        ixy="0.0"
+        ixz="0.0"
+        iyy="0.0001"
+        iyz="0.0"
+        izz="0.0001" />
     </inertial>
     <visual>
@@ -423,5 +423,5 @@
     type="fixed">
     <origin
-      xyz="-0.245 0 -0.04"
+      xyz="-0.245 0 -0.0384"
       rpy="0 0 0" />
     <parent

File: src/smrr_description/urdf/test.urdf.xacro (robot description, xacro)
@@ -9,4 +9,5 @@
     <xacro:include filename="$(find smrr_description)/urdf/camera.urdf.xacro" />
     <xacro:include filename="$(find smrr_description)/urdf/lidar.urdf.xacro" />
+    <!-- <xacro:include filename="$(find smrr_description)/urdf/imu.urdf.xacro" /> -->
     <xacro:include filename="$(find smrr_description)/urdf/transmission.urdf.xacro" />
     <xacro:include filename="$(find smrr_description)/urdf/smrr_ros2_control.urdf.xacro" />

Commit message: Added the outside elevator up and down

File: src/smrr_description/urdf/camera.urdf.xacro (robot description, xacro)
@@ -2,5 +2,5 @@
 <robot xmlns:xacro="http://www.ros.org/wiki/xacro">
     <joint name="camera_joint" type="fixed">
-        <origin xyz="0.06 0 1.1" rpy="0 0 0"/>
+        <origin xyz="0.055 0 1.2174" rpy="0 0 0"/>
         <parent link="base_link"/>
         <child link="camera_link"/>

Commit message: Refactor code structure for improved readability and maintainability

File: src/smrr_description/urdf/camera.urdf.xacro (robot description, xacro)
@@ -2,5 +2,5 @@
 <robot xmlns:xacro="http://www.ros.org/wiki/xacro">
     <joint name="camera_joint" type="fixed">
-        <origin xyz="0.06 0 1.1" rpy="0 0 0"/>
+        <origin xyz="0.06 0.012 1.1974" rpy="0 -0.10472 0"/>
         <parent link="base_link"/>
         <child link="camera_link"/>

File: src/smrr_description/urdf/lidar.urdf.xacro (robot description, xacro)
@@ -23,5 +23,5 @@
     </link>
 	<joint name="rplidar_joint" type="fixed">
-		<origin xyz="0.24 0  0.1874" rpy="0 0 0 "/>
+		<origin xyz="0.1704 0  0.1874" rpy="0 0 0 "/>
 		<parent link="base_link"/>
 		<child link="rplidar_link"/>

File: src/smrr_description/urdf/mobile_base.urdf.xacro (robot description, xacro)
@@ -347,3 +347,9 @@
       xyz="1 0 0" />
   </joint>
+  <link name="link_0_fake"/>
+  <joint name="link_0_fake_joint" type="fixed">
+    <origin xyz="-0.04 -0.235 1.11974" rpy="0 0 0"/>
+    <parent link="base_link"/>
+    <child  link="link_0_fake"/>
+  </joint>
 </robot>

Commit message: Update SLLIDAR submodule, modify launch files, adjust camera URDF, and refine docking configuration
- Updated SLLIDAR submodule to a dirty state.
- Commented out the human tracker group in the smrr.launch.py file.
- Adjusted the rear camera joint position in camera.urdf.xacro for better alignment.
- Increased wait charge timeout and adjusted undock/rotation angular tolerances in docking.yaml.
- Modified docking behavior parameters including docking threshold and staging pose offsets.
- Updated camera topic and info topic in detections.launch.py to use the rear camera.
- Changed the position of the dock link in detections.launch.py for better alignment.
- Removed redundant QoS settings in docking_bringup_hardware.launch.py and adjusted camera frame parameters.

File: src/smrr_description/urdf/camera.urdf.xacro (robot description, xacro)
@@ -141,5 +141,5 @@
     <!-- Rear Camera Mount (facing backward for docking) -->
     <joint name="rear_camera_joint" type="fixed">
-        <origin xyz="-0.12 0 0.43" rpy="0 0 ${pi}"/>  <!-- Mounted at back, rotated 180° -->
+        <origin xyz="-0.12 0 0.3524" rpy="0 0 ${pi}"/>  <!-- Mounted at back, rotated 180° -->
         <parent link="base_link"/>
         <child link="rear_camera_link"/>
