Commit message: Selective merge from robot-branch + simulation fixes
- Merged non-hardware packages from upstream/robot-branch:
  smrr_base_controller, smrr_bringup, smrr_controller (hardware_controller),
  smrr_description (urdf/lidar/ros2_control), smrr_docking, smrr_human_tracker,
  smrr_navigation (elevator_call_button_server, hardware launch/maps),
  smrr_rectify (new package)

- Excluded hardware-specific packages: zed2, sllidar_ros2
- Excluded hardware-specific configs: camera.urdf.xacro, zed_override.yaml,
  zed_topic_restamper.py, laser_scan_240deg_filter.yaml, arm_controller.yaml,
  modified_ekf.yaml (kept at 9acd1a2 for simulation compatibility)
- Removed zed_topic_restamper.py from smrr_bringup CMakeLists.txt install target
- Fixed MPPI GoalAngleCritic weight (6.0->2.0) and threshold (0.25->0.50m)
  to prevent post-goal rotation oscillation in simulation

File: src/smrr_description/urdf/smrr_ros2_control.urdf.xacro (robot description, xacro)
@@ -3,83 +3,83 @@
   <xacro:property name="PI" value="3.14159265359" />
   <xacro:arg name="is_sim" default="true"/>
-  <ros2_control name="RobotSystem" type="system">
-    <!-- ros2_control Simulated Robot -->
-    <xacro:if value="$(arg is_sim)">
-      <hardware>
-        <plugin>gazebo_ros2_control/GazeboSystem</plugin>
-      </hardware>
-      <joint name="shoulder_r_joint">
-        <command_interface name="position">
-          <param name="min">0</param>
-          <param name="max">${0.5*PI}</param>
-        </command_interface>
-        <!-- <command_interface name="velocity">
-          <param name="min">-3.14</param>
-          <param name="max">3.14</param>
-        </command_interface> -->
-        <state_interface name="position"/>
-        <!-- <state_interface name="velocity"/> -->
-      </joint>
-      <joint name="bicep_r_joint">
-        <command_interface name="position">
-          <param name="min">${-0.25*PI}</param>
-          <param name="max">${0.25*PI}</param>
-        </command_interface>
-        <!-- <command_interface name="velocity">
-          <param name="min">-3.14</param>
-          <param name="max">3.14</param>
-        </command_interface> -->
-        <state_interface name="position"/>
-        <!-- <state_interface name="velocity"/> -->
-      </joint>
-      <joint name="elbow_r_joint">
-        <command_interface name="position">
-          <param name="min">0</param>
-          <param name="max">${0.5*PI}</param>
-        </command_interface>
-        <!-- <command_interface name="velocity">
-          <param name="min">-3.14</param>
-          <param name="max">3.14</param>
-        </command_interface> -->
-        <state_interface name="position"/>
-        <!-- <state_interface name="velocity"/> -->
-      </joint>
-      <joint name="wrist_r_joint">
-        <command_interface name="position">
-          <param name="min">${-0.25*PI}</param>
-          <param name="max">${0.25*PI}</param>
-        </command_interface>
-        <!-- <command_interface name="velocity">
-          <param name="min">-3.14</param>
-          <param name="max">3.14</param>
-        </command_interface> -->
-        <state_interface name="position"/>
-        <!-- <state_interface name="velocity"/> -->
-      </joint>
-    </xacro:if>
-    <!-- ros2_control Real Robot -->
-    <xacro:unless value="$(arg is_sim)">
-      <hardware>
-        <plugin>smrr_base_controller/BaseController</plugin>
-        <param name="port">/dev/ttyUSB0</param>
-        <!-- /dev/ttyACM0 -->
-      </hardware>
-    </xacro:unless>
-    <joint name="left_wheel_joint">
-      <command_interface name="velocity">
-        <param name="min">-10</param>
-        <param name="max">10</param>
-      </command_interface>
-      <state_interface name="position"/>
-      <state_interface name="velocity"/>
-    </joint>
-    <joint name="right_wheel_joint">
-      <command_interface name="velocity">
-        <param name="min">-10</param>
-        <param name="max">10</param>
-      </command_interface>
-      <state_interface name="position"/>
-      <state_interface name="velocity"/>
-    </joint>
-  </ros2_control>
+    <ros2_control name="RobotSystem" type="system">
+        <!-- ros2_control Simulated Robot -->
+        <xacro:if value="$(arg is_sim)">
+            <hardware>
+                <plugin>gazebo_ros2_control/GazeboSystem</plugin>
+            </hardware>
+        </xacro:if>
+        <!-- ros2_control Real Robot -->
+        <xacro:unless value="$(arg is_sim)">
+            <hardware>
+                <plugin>smrr_base_controller/BaseController</plugin>
+                <param name="port">/dev/ttyACM1</param>
+                <!-- /dev/ttyUSB0 -->
+            </hardware>
+        </xacro:unless>
+        <joint name="shoulder_r_joint">
+            <command_interface name="position">
+              <param name="min">0</param>
+              <param name="max">${0.5*PI}</param>
+            </command_interface>
+            <!-- <command_interface name="velocity">
+              <param name="min">-3.14</param>
+              <param name="max">3.14</param>
+            </command_interface> -->
+            <state_interface name="position"/>
+            <!-- <state_interface name="velocity"/> -->
+        </joint>
+        <joint name="bicep_r_joint">
+            <command_interface name="position">
+              <param name="min">${-0.25*PI}</param>
+              <param name="max">${0.25*PI}</param>
+            </command_interface>
+            <!-- <command_interface name="velocity">
+              <param name="min">-3.14</param>
+              <param name="max">3.14</param>
+            </command_interface> -->
+            <state_interface name="position"/>
+            <!-- <state_interface name="velocity"/> -->
+        </joint>
+        <joint name="elbow_r_joint">
+            <command_interface name="position">
+              <param name="min">0</param>
+              <param name="max">${0.5*PI}</param>
+            </command_interface>
+            <!-- <command_interface name="velocity">
+              <param name="min">-3.14</param>
+              <param name="max">3.14</param>
+            </command_interface> -->
+            <state_interface name="position"/>
+            <!-- <state_interface name="velocity"/> -->
+        </joint>
+        <joint name="wrist_r_joint">
+            <command_interface name="position">
+              <param name="min">${-0.25*PI}</param>
+              <param name="max">${0.25*PI}</param>
+            </command_interface>
+            <!-- <command_interface name="velocity">
+              <param name="min">-3.14</param>
+              <param name="max">3.14</param>
+            </command_interface> -->
+            <state_interface name="position"/>
+            <!-- <state_interface name="velocity"/> -->
+        </joint>
+        <joint name="left_wheel_joint">
+            <command_interface name="velocity">
+                <param name="min">-10</param>
+                <param name="max">10</param>
+            </command_interface>
+            <state_interface name="position"/>
+            <state_interface name="velocity"/>
+        </joint>
+        <joint name="right_wheel_joint">
+            <command_interface name="velocity">
+                <param name="min">-10</param>
+                <param name="max">10</param>
+            </command_interface>
+            <state_interface name="position"/>
+            <state_interface name="velocity"/>
+        </joint>
+    </ros2_control>
 </robot>

File: src/smrr_description/urdf/test.urdf.xacro (robot description, xacro)
@@ -9,7 +9,12 @@
     <xacro:include filename="$(find smrr_description)/urdf/camera.urdf.xacro" />
     <xacro:include filename="$(find smrr_description)/urdf/lidar.urdf.xacro" />
-    <!-- <xacro:include filename="$(find smrr_description)/urdf/imu.urdf.xacro" /> -->
     <xacro:include filename="$(find smrr_description)/urdf/transmission.urdf.xacro" />
-    <xacro:include filename="$(find smrr_description)/urdf/smrr_ros2_control.urdf.xacro" />
+    <!-- Use different ros2_control config for sim vs hardware -->
+    <xacro:if value="$(arg is_sim)">
+        <xacro:include filename="$(find smrr_description)/urdf/smrr_ros2_control.urdf.xacro" />
+    </xacro:if>
+    <xacro:unless value="$(arg is_sim)">
+        <xacro:include filename="$(find smrr_description)/urdf/smrr_ros2_control_hardware.urdf.xacro" />
+    </xacro:unless>
     <xacro:include filename="$(find smrr_description)/urdf/gazebo_ros2_control.urdf.xacro" />
 </robot>
