Commit message: Updated the robot description urdf with the docking part in the mobile base. Tuned the navigation parameters.

File: src/smrr_description/urdf/mobile_base.urdf.xacro (robot description, xacro)
@@ -203,4 +203,90 @@
       <dynamics damping="0.3" friction="0.5"/>
   </joint>
+  <!-- <link
+    name="docking_station_mount">
+    <inertial>
+      <origin
+        xyz="2.46415216024198E-05 -0.0079159646726803 0.0969814867787446"
+        rpy="0 0 0" />
+      <mass
+        value="0.312805817268065" />
+      <inertia
+        ixx="0.000884962592461685"
+        ixy="3.85178154688985E-07"
+        ixz="4.77831152807354E-07"
+        iyy="0.00125523278460193"
+        iyz="-0.000141824356047521"
+        izz="0.00151275866886532" />
+    </inertial>
+    <visual>
+      <origin
+        xyz="0 0 0"
+        rpy="0 0 0" />
+      <geometry>
+        <mesh
+          filename="package://smrr_description/meshes/Docking_assembly.STL"
+          scale="0.001 0.001 0.001" />
+      </geometry>
+      <material
+        name="docking_grey">
+        <color
+          rgba="0.792156862745098 0.819607843137255 0.933333333333333 1" />
+      </material>
+    </visual>
+    <collision>
+      <origin
+        xyz="0 0 0"
+        rpy="0 0 0" />
+      <geometry>
+        <mesh
+          filename="package://smrr_description/meshes/Docking_assembly.STL"
+          scale="0.001 0.001 0.001" />
+      </geometry>
+    </collision>
+  </link>
+  <joint
+    name="docking_mount_joint"
+    type="fixed">
+    <origin
+      xyz="-0.14469 -2.0850 0.46748"
+      rpy="3.1416 1.5708 0" />
+    <parent
+      link="base_link" />
+    <child
+      link="docking_station_mount" />
+    <axis
+      xyz="0 0 0" />
+  </joint> -->
+      <link name="docking_station_mount">
+    <inertial>
+      <origin xyz="2.46415216024198e-05 -0.0079159646726803 0.0969814867787446" rpy="0 0 0"/>
+      <mass value="0.312805817268065"/>
+      <inertia ixx="0.000884962592461685" ixy="3.85178154688985e-07" ixz="4.77831152807354e-07"
+               iyy="0.00125523278460193" iyz="-0.000141824356047521" izz="0.00151275866886532"/>
+    </inertial>
+    <visual>
+      <origin xyz="-0.41401 -0.9544 -0.96557" rpy="0 0 0"/>
+      <geometry>
+        <!-- keep your current mesh and scale; change only if your asset uses meters already -->
+        <mesh filename="package://smrr_description/meshes/Docking_assembly.STL" scale="0.001 0.001 0.001"/>
+      </geometry>
+      <material name="docking_grey">
+        <color rgba="0.7921568627 0.8196078431 0.9333333333 1"/>
+      </material>
+    </visual>
+    <collision>
+      <origin xyz="-0.41401 -0.9544 -0.96557" rpy="0 0 0"/>
+      <geometry>
+        <mesh filename="package://smrr_description/meshes/Docking_assembly.STL" scale="0.001 0.001 0.001"/>
+      </geometry>
+    </collision>
+  </link>
+  <joint name="docking_mount_joint" type="fixed">
+    <!-- docking pose from SolidWorks, transformed into your base_link using wheel joints as anchors -->
+    <origin xyz="-0.275 0 0" rpy="0 0 0"/>
+    <parent link="base_link"/>
+    <child  link="docking_station_mount"/>
+    <axis xyz="0 0 0"/>
+  </joint>
   <link
     name="front_caster">

File: src/smrr_description/urdf/smrr_ros2_control.urdf.xacro (robot description, xacro)
@@ -3,83 +3,83 @@
   <xacro:property name="PI" value="3.14159265359" />
   <xacro:arg name="is_sim" default="true"/>
-    <ros2_control name="RobotSystem" type="system">
-        <!-- ros2_control Simulated Robot -->
-        <xacro:if value="$(arg is_sim)">
-            <hardware>
-                <plugin>gazebo_ros2_control/GazeboSystem</plugin>
-            </hardware>
-        </xacro:if>
-        <!-- ros2_control Real Robot -->
-        <xacro:unless value="$(arg is_sim)">
-            <hardware>
-                <plugin>smrr_base_controller/BaseController</plugin>
-                <param name="port">/dev/ttyUSB0</param>
-                <!-- /dev/ttyACM0 -->
-            </hardware>
-        </xacro:unless>
-        <joint name="shoulder_r_joint">
-            <command_interface name="position">
-              <param name="min">0</param>
-              <param name="max">${0.5*PI}</param>
-            </command_interface>
-            <!-- <command_interface name="velocity">
-              <param name="min">-3.14</param>
-              <param name="max">3.14</param>
-            </command_interface> -->
-            <state_interface name="position"/>
-            <!-- <state_interface name="velocity"/> -->
-        </joint>
-        <joint name="bicep_r_joint">
-            <command_interface name="position">
-              <param name="min">${-0.25*PI}</param>
-              <param name="max">${0.25*PI}</param>
-            </command_interface>
-            <!-- <command_interface name="velocity">
-              <param name="min">-3.14</param>
-              <param name="max">3.14</param>
-            </command_interface> -->
-            <state_interface name="position"/>
-            <!-- <state_interface name="velocity"/> -->
-        </joint>
-        <joint name="elbow_r_joint">
-            <command_interface name="position">
-              <param name="min">0</param>
-              <param name="max">${0.5*PI}</param>
-            </command_interface>
-            <!-- <command_interface name="velocity">
-              <param name="min">-3.14</param>
-              <param name="max">3.14</param>
-            </command_interface> -->
-            <state_interface name="position"/>
-            <!-- <state_interface name="velocity"/> -->
-        </joint>
-        <joint name="wrist_r_joint">
-            <command_interface name="position">
-              <param name="min">${-0.25*PI}</param>
-              <param name="max">${0.25*PI}</param>
-            </command_interface>
-            <!-- <command_interface name="velocity">
-              <param name="min">-3.14</param>
-              <param name="max">3.14</param>
-            </command_interface> -->
-            <state_interface name="position"/>
-            <!-- <state_interface name="velocity"/> -->
-        </joint>
-        <joint name="left_wheel_joint">
-            <command_interface name="velocity">
-                <param name="min">-10</param>
-                <param name="max">10</param>
-            </command_interface>
-            <state_interface name="position"/>
-            <state_interface name="velocity"/>
-        </joint>
-        <joint name="right_wheel_joint">
-            <command_interface name="velocity">
-                <param name="min">-10</param>
-                <param name="max">10</param>
-            </command_interface>
-            <state_interface name="position"/>
-            <state_interface name="velocity"/>
-        </joint>
-    </ros2_control>
+  <ros2_control name="RobotSystem" type="system">
+    <!-- ros2_control Simulated Robot -->
+    <xacro:if value="$(arg is_sim)">
+      <hardware>
+        <plugin>gazebo_ros2_control/GazeboSystem</plugin>
+      </hardware>
+      <joint name="shoulder_r_joint">
+        <command_interface name="position">
+          <param name="min">0</param>
+          <param name="max">${0.5*PI}</param>
+        </command_interface>
+        <!-- <command_interface name="velocity">
+          <param name="min">-3.14</param>
+          <param name="max">3.14</param>
+        </command_interface> -->
+        <state_interface name="position"/>
+        <!-- <state_interface name="velocity"/> -->
+      </joint>
+      <joint name="bicep_r_joint">
+        <command_interface name="position">
+          <param name="min">${-0.25*PI}</param>
+          <param name="max">${0.25*PI}</param>
+        </command_interface>
+        <!-- <command_interface name="velocity">
+          <param name="min">-3.14</param>
+          <param name="max">3.14</param>
+        </command_interface> -->
+        <state_interface name="position"/>
+        <!-- <state_interface name="velocity"/> -->
+      </joint>
+      <joint name="elbow_r_joint">
+        <command_interface name="position">
+          <param name="min">0</param>
+          <param name="max">${0.5*PI}</param>
+        </command_interface>
+        <!-- <command_interface name="velocity">
+          <param name="min">-3.14</param>
+          <param name="max">3.14</param>
+        </command_interface> -->
+        <state_interface name="position"/>
+        <!-- <state_interface name="velocity"/> -->
+      </joint>
+      <joint name="wrist_r_joint">
+        <command_interface name="position">
+          <param name="min">${-0.25*PI}</param>
+          <param name="max">${0.25*PI}</param>
+        </command_interface>
+        <!-- <command_interface name="velocity">
+          <param name="min">-3.14</param>
+          <param name="max">3.14</param>
+        </command_interface> -->
+        <state_interface name="position"/>
+        <!-- <state_interface name="velocity"/> -->
+      </joint>
+    </xacro:if>
+    <!-- ros2_control Real Robot -->
+    <xacro:unless value="$(arg is_sim)">
+      <hardware>
+        <plugin>smrr_base_controller/BaseController</plugin>
+        <param name="port">/dev/ttyUSB0</param>
+        <!-- /dev/ttyACM0 -->
+      </hardware>
+    </xacro:unless>
+    <joint name="left_wheel_joint">
+      <command_interface name="velocity">
+        <param name="min">-10</param>
+        <param name="max">10</param>
+      </command_interface>
+      <state_interface name="position"/>
+      <state_interface name="velocity"/>
+    </joint>
+    <joint name="right_wheel_joint">
+      <command_interface name="velocity">
+        <param name="min">-10</param>
+        <param name="max">10</param>
+      </command_interface>
+      <state_interface name="position"/>
+      <state_interface name="velocity"/>
+    </joint>
+  </ros2_control>
 </robot>

File: src/smrr_description/urdf/test.urdf.xacro (robot description, xacro)
@@ -10,11 +10,5 @@
     <xacro:include filename="$(find smrr_description)/urdf/lidar.urdf.xacro" />
     <xacro:include filename="$(find smrr_description)/urdf/transmission.urdf.xacro" />
-    <!-- Use different ros2_control config for sim vs hardware -->
-    <xacro:if value="$(arg is_sim)">
-        <xacro:include filename="$(find smrr_description)/urdf/smrr_ros2_control.urdf.xacro" />
-    </xacro:if>
-    <xacro:unless value="$(arg is_sim)">
-        <xacro:include filename="$(find smrr_description)/urdf/smrr_ros2_control_hardware.urdf.xacro" />
-    </xacro:unless>
+    <xacro:include filename="$(find smrr_description)/urdf/smrr_ros2_control.urdf.xacro" />
     <xacro:include filename="$(find smrr_description)/urdf/gazebo_ros2_control.urdf.xacro" />
 </robot>

Commit message: Update the multifloor navogation algorithm to use only one map per floor.

File: src/smrr_description/urdf/mobile_base.urdf.xacro (robot description, xacro)
@@ -17,17 +17,15 @@
     <inertial>
       <origin
-        xyz="0.0201310485852864 0.000520829416461865 0.865026738420884"
-        rpy="0 0 0" />
-      <mass
-        value="8.2797481488828" /> <!-- 28.2797481488828 -->
-      <!-- <mass
-        value="48.2797481488828" /> -->
-      <inertia
-        ixx="1.40869842198577"
-        ixy="0.00172519109922957"
-        ixz="0.0295451682055194"
-        iyy="1.38963154057563"
-        iyz="-0.00609490500279897"
-        izz="0.244482664433787" />
+        xyz="0.0201310485852864 0.000520829416461865 0.35"
+        rpy="0 0 0" />
+      <mass
+        value="17.0" />
+      <inertia
+        ixx="1.5"
+        ixy="0.0"
+        ixz="0.0"
+        iyy="1.5"
+        iyz="0.0"
+        izz="1.0" />
     </inertial>
     <visual>
@@ -126,5 +124,5 @@
     <axis
       xyz="0 0 1" />
-    <dynamics damping="0.3" friction="0.5"/>
+    <dynamics damping="0.1" friction="0.01"/>
   </joint>
   <link
@@ -201,5 +199,5 @@
       <axis
         xyz="0 0 1" />
-      <dynamics damping="0.3" friction="0.5"/>
+      <dynamics damping="0.1" friction="0.01"/>
   </joint>
   <!-- <link
@@ -360,4 +358,5 @@
     <axis
       xyz="1 0 0" />
+    <dynamics damping="0.0" friction="0.0"/>
   </joint>
   <link
@@ -432,4 +431,5 @@
     <axis
       xyz="1 0 0" />
+    <dynamics damping="0.0" friction="0.0"/>
   </joint>
 </robot>

Commit message: Updated with the spencer architecure for the perception pipeline.

File: src/smrr_description/urdf/mobile_base.urdf.xacro (robot description, xacro)
@@ -273,10 +273,4 @@
       </material>
     </visual>
-    <collision>
-      <origin xyz="-0.41401 -0.9544 -0.96557" rpy="0 0 0"/>
-      <geometry>
-        <mesh filename="package://smrr_description/meshes/Docking_assembly.STL" scale="0.001 0.001 0.001"/>
-      </geometry>
-    </collision>
   </link>
   <joint name="docking_mount_joint" type="fixed">
@@ -350,5 +344,5 @@
     type="fixed">
     <origin
-      xyz="0.245 0 -0.0414"
+      xyz="0.245 0 -0.0384"
       rpy="0 0 0" />
     <parent
@@ -356,6 +350,5 @@
     <child
       link="front_caster" />
-    <axis
-      xyz="1 0 0" />
+    <axis xyz="0 1 0" />
     <dynamics damping="0.0" friction="0.0"/>
   </joint>
@@ -429,6 +422,5 @@
     <child
       link="back_caster" />
-    <axis
-      xyz="1 0 0" />
+    <axis xyz="0 1 0" />
     <dynamics damping="0.0" friction="0.0"/>
   </joint>

File: src/smrr_description/urdf/transmission.urdf.xacro (robot description, xacro)
@@ -75,5 +75,5 @@
     </gazebo>
     <gazebo reference="right_wheel">
-        <mu1>1000000.0</mu1>  <!--1000000000000000.0-->
+        <mu1>100000.0</mu1>  <!--1000000000000000.0-->
         <mu2>1000000.0</mu2>
         <minDepth>0.005</minDepth>
@@ -88,12 +88,12 @@
     </gazebo>
     <gazebo reference="front_caster">
-        <mu1>0.1</mu1>
-        <mu2>0.1</mu2>
+        <mu1>0.0</mu1>
+        <mu2>0.0</mu2>
         <minDepth>0.005</minDepth>
         <!-- 0.002 -->
     </gazebo>
     <gazebo reference="back_caster">
-        <mu1>0.1</mu1>
-        <mu2>0.1</mu2>
+        <mu1>0.0</mu1>
+        <mu2>0.0</mu2>
         <minDepth>0.005</minDepth>
     </gazebo>

Commit message: Updated the floor arrival detection with the new model button-detection.pt and added the link_0_fake for right hand.

File: src/smrr_description/urdf/mobile_base.urdf.xacro (robot description, xacro)
@@ -425,3 +425,9 @@
     <dynamics damping="0.0" friction="0.0"/>
   </joint>
+  <link name="link_0_fake"/>
+  <joint name="link_0_fake_joint" type="fixed">
+    <origin xyz="-0.04 -0.225 1.2174" rpy="0 0 0"/>
+    <parent link="base_link"/>
+    <child  link="link_0_fake"/>
+  </joint>
 </robot>

Commit message: Updated the up and down button pressing service elevator to have specific offsets depending on the button that's going to press.

File: src/smrr_description/urdf/mobile_base.urdf.xacro (robot description, xacro)
@@ -349,5 +349,6 @@
   <link name="link_0_fake"/>
   <joint name="link_0_fake_joint" type="fixed">
-    <origin xyz="-0.04 -0.235 1.11974" rpy="0 0 0"/>
+    <!-- <origin xyz="-0.05799 -0.21910 1.18100" rpy="0.01475 -0.01943 -0.07311"/> -->
+    <origin xyz="-0.04869 -0.21265 1.21385" rpy="-0.00434 0.02883 -0.08261"/>
     <parent link="base_link"/>
     <child  link="link_0_fake"/>

Commit message: Working docking updates

File: src/smrr_description/urdf/mobile_base.urdf.xacro (robot description, xacro)
@@ -349,6 +349,7 @@
   <link name="link_0_fake"/>
   <joint name="link_0_fake_joint" type="fixed">
-    <!-- <origin xyz="-0.05799 -0.21910 1.18100" rpy="0.01475 -0.01943 -0.07311"/> -->
-    <origin xyz="-0.04869 -0.21265 1.21385" rpy="-0.00434 0.02883 -0.08261"/>
+    <!-- <origin xyz="-0.056947 -0.216501 1.178662" rpy="0.009267 -0.023331 -0.076002"/> old-->
+    <!-- <origin xyz="-0.04869 -0.21265 1.21385" rpy="-0.00434 0.02883 -0.08261"/> -->
+    <origin xyz="-0.06173 -0.20542 1.20073" rpy="0.04485 0.06728 -0.05866"/>
     <parent link="base_link"/>
     <child  link="link_0_fake"/>
